File: pcb/kickswitch.sch (KiCad schematic (older format))
At the start: 4 parts, among them U1 4075, U2 4081

Commit message: Added NET file and component library
Parts:
- gave numbers to parts that had none: 1
Connections:
- wire segments 59 -> 43
Changed lines of the file:
@@
 LIBS:valves
 LIBS:cmos_ieee
-LIBS:kickswitch-cache
+LIBS:ROMs
 EELAYER 25 0
 EELAYER END
@@
 $EndComp
 Wire Wire Line
-	800  5700 1050 5700
-Wire Wire Line
-	1050 5700 1950 5700
-Wire Wire Line
-	1950 5700 5450 5700
+	800  5700 5450 5700
 $Comp
-L GND #PWR?
+L GND #PWR1
 U 1 1 5AF89539
 P 800 5700
-F 0 "#PWR?" H 800 5450 50  0001 C CNN
+F 0 "#PWR1" H 800 5450 50  0001 C CNN
 F 1 "GND" H 800 5550 50  0000 C CNN
 F 2 "" H 800 5700 50  0001 C CNN
@@
 $EndComp
 $Comp
-L Conn_01x07 J?
+L Conn_01x07 J1
 U 1 1 5AF89555
 P 800 3350
-F 0 "J?" H 800 3750 50  0000 C CNN
+F 0 "J1" H 800 3750 50  0000 C CNN
 F 1 "Conn_01x07" H 800 2950 50  0000 C CNN
 F 2 "" H 800 3350 50  0001 C CNN
@@
 $EndComp
 Wire Wire Line
-	950  2550 1200 2550
-Wire Wire Line
-	1200 2550 1200 2550
-Wire Wire Line
-	1200 2550 5350 2550
+	950  2550 5350 2550
 Wire Wire Line
 	1200 2550 1200 3050
@@
 Connection ~ 1200 2550
 Wire Wire Line
-	1000 3550 1200 3550
-Wire Wire Line
-	1200 3550 2050 3550
+	1000 3550 2050 3550
 Wire Wire Line
 	2050 3550 2050 5200
 Wire Wire Line
-	1000 3650 1150 3650
+	1000 3650 1950 3650
 Wire Wire Line
-	1150 3650 1950 3650
-Wire Wire Line
-	1950 3650 1950 3900
-Wire Wire Line
-	1950 3900 1950 5300
+	1950 3650 1950 5300
 Wire Wire Line
 	1950 5300 2050 5300
@@
 Connection ~ 1950 5700
 Wire Wire Line
-	3050 5300 3100 5300
-Wire Wire Line
-	3100 5300 5450 5300
+	3050 5300 5450 5300
 Text Label 5250 5250 0    60   ~ 0
 A19
@@
 	2550 3250 2550 4350
 Wire Wire Line
-	1000 3250 1350 3250
-Wire Wire Line
-	1350 3250 2550 3250
+	1000 3250 2550 3250
 Wire Wire Line
 	4300 4450 2450 4450
 Wire Wire Line
-	1000 3450 1250 3450
-Wire Wire Line
-	1250 3450 2450 3450
-Wire Wire Line
-	2450 3450 2900 3450
+	1000 3450 2900 3450
 Wire Wire Line
 	4300 4950 4300 4550
@@
 	2450 4450 2450 3450
 Wire Wire Line
-	1000 3350 1300 3350
-Wire Wire Line
-	1300 3350 3050 3350
+	1000 3350 3050 3350
 Wire Wire Line
 	3050 3350 3050 3700
@@
 S   ?   ?  p1\nR  p42 p1  p2\n   A19 A18 A17\ni1  0   0   0\ni2  0   0   1\ni3  0   1   0\ni4  0   1   1\ni5  1   0   x\ni6  1   1   x\n\nA19 = (i5 | i6)\nA18 = (i3 | i4) | i6\nA17 = (i2 | i4) | (A19 & a17[in])\n\n\n\nPin 31 high - already provided by socket?\n4.7kohm pullups on address pins? maybe not needed.
 $Comp
-L VCC #PWR?
+L VCC #PWR2
 U 1 1 5B090894
 P 950 2550
-F 0 "#PWR?" H 950 2400 50  0001 C CNN
+F 0 "#PWR2" H 950 2400 50  0001 C CNN
 F 1 "VCC" H 950 2700 50  0000 C CNN
 F 2 "" H 950 2550 50  0001 C CNN
@@
 	1350 4200 1050 4200
 Wire Wire Line
-	1050 4200 1050 4500
-Wire Wire Line
-	1050 4500 1050 4800
-Wire Wire Line
-	1050 4800 1050 5100
-Wire Wire Line
-	1050 5100 1050 5400
-Wire Wire Line
-	1050 5400 1050 5700
+	1050 4200 1050 5700
 Connection ~ 1050 5700
 Wire Wire Line

Commit message: Latest version. Added Arduino code
Parts:
- removed J1: Conn_01x07, symbol Conn_01x07
- removed RN1: R_Pack05_SIP, Resistors_THT:R_Array_SIP10, symbol R_Pack05_SIP
- removed U1: 4075, symbol 4075
- removed U2: 4081, symbol 4081
- added C1, C2: 22pf, Capacitors_SMD:C_0603, symbol C_Small
- added C3: 100nF, Capacitors_SMD:C_0603, symbol C_Small
- added D1: 1n4148, Diodes_SMD:D_SOD-123F, symbol D
- added J2: 2x4hdr, Pin_Headers:Pin_Header_Straight_2x04_Pitch2.54mm, symbol Conn_02x04_Odd_Even
- added R1: 10k, Resistors_SMD:R_0603, symbol R
- added SW1: SW_RST, Buttons_Switches_SMD:SW_SPST_B3S-1000, symbol SW_Push
- added U1: SN74LVC1G08, TO_SOT_Packages_SMD:SOT-23-5, symbol SN74LVC1G08
- added U2: SN74LVC1G32, TO_SOT_Packages_SMD:SOT-23-5, symbol SN74LVC1G32
- added U3: ATMEGA328P-PU, Housings_DIP:DIP-28_W7.62mm, symbol ATMEGA328P-PU
- added U4: MC23C4100_socket, Housings_DIP:DIP-40_W15.24mm_Socket, symbol MC23C4100_socket
- added U5: M27C160, Housings_DIP:DIP-42_W15.24mm_Socket, symbol M27C160
- added Y1: 16MHz, Crystals:Crystal_HC49-4H_Vertical, symbol Crystal
Connections:
- net labels added: A0, A1, A10, A11, A12, A13, A14, A15, A16, A17_orig, A17_set, A17in, A17out, A18_set, A18out, A19_set, A19out, A2, A3, A4, A5, A6, A7, A8, A9, D0, D1, D10, D11, D12, D13, D14, D15, D2, D3, D4, D5, D6, D7, D8, D9, Gnd, MISO, MOSI, RESET, RXD, SCK, TXD, Vcc
- net labels removed: A17, A17_in, A18, A19, GND, VCC
- wire segments 43 -> 177
- no-connect marks 0 -> 15
Other:
- note removed: "S ? ? p1\nR p42 p1 p2\n A19 A18 A17\ni1 0 0 0\ni2 0 0 1\ni3 0 1 0\ni4 0 1 1\ni5 1 0 x\ni6 1 1 x\n\nA19 = (i5 | i6)\nA18 = (i3 | i4) | i6\nA17 = (i2 | i4) | (A19 & a17[in])\n\n\n\nPin 31 high - already provided by socket?\n4.7kohm pullups on address pins? maybe not needed."

Commit message: Added many more I/O pins Removed reset button Added resistor nets for Address line pullups Added ground plane
Parts:
- removed J2: 2x4hdr, Pin_Headers:Pin_Header_Straight_2x04_Pitch2.54mm, symbol Conn_02x04_Odd_Even
- removed SW1: SW_RST, Buttons_Switches_SMD:SW_SPST_B3S-1000, symbol SW_Push
- added J1: Conn_02x10_Odd_Even, Pin_Headers:Pin_Header_Straight_2x10_Pitch2.54mm, symbol Conn_02x10_Odd_Even
- added RN1: 4k7, Resistors_THT:R_Array_SIP9, symbol R_Network08
- added RN2: 4k7, Resistors_THT:R_Array_SIP10, symbol R_Network09
Connections:
- net labels added: AREF, PB0, PB1, PB2, PC4, PC5, PD2, PD3, PD4, PD5, PD6, PD7, ~RESET
- net labels removed: A18out, A19out, RESET
- wire segments 177 -> 248
- no-connect marks 15 -> 2
Other:
- moved on the sheet: C1, C2, C3, D1, R1, U1, U2, U3, U4, U5, Y1

Commit message: Upgraded to latest KiCAD. Eliminated encoder. Eliminated switch and added /RSTOUT input line instead. Added jumper for pin 1/31 "Oops" fix. Updated README.md.
Parts:
- added J2: Conn_01x03, Pin_Headers:Pin_Header_Straight_1x03_Pitch2.54mm, symbol Connector_Generic:Conn_01x03
- C1, C2, C3: symbol C_Small -> kickswitch-rescue:C_Small
- D1: symbol D -> kickswitch-rescue:D
- J1: symbol Conn_02x10_Odd_Even -> kickswitch-rescue:Conn_02x10_Odd_Even
- R1: symbol R -> kickswitch-rescue:R
- RN1: symbol R_Network08 -> kickswitch-rescue:R_Network08
- RN2: symbol R_Network09 -> kickswitch-rescue:R_Network09
- U1: symbol SN74LVC1G08 -> kickswitch-rescue:SN74LVC1G08
- U2: symbol SN74LVC1G32 -> kickswitch-rescue:SN74LVC1G32
- U3: symbol ATMEGA328P-PU -> kickswitch-rescue:ATMEGA328P-PU
- U4: symbol MC23C4100_socket -> kickswitch-rescue:MC23C4100_socket
- U5: symbol M27C160 -> kickswitch-rescue:M27C160
- Y1: symbol Crystal -> kickswitch-rescue:Crystal
Connections:
- net A17in: now also J2.2 (Pin_2); no longer U4.31 (A17)
- net at U4.1 (Oops): now also J2.1 (Pin_1)
- new net: J2.3 (Pin_3), U4.31 (A17)
- no-connect marks 2 -> 1
Changed lines of the file:
@@
-EESchema Schematic File Version 2
-LIBS:power
-LIBS:device
-LIBS:switches
-LIBS:relays
-LIBS:motors
-LIBS:transistors
-LIBS:conn
-LIBS:linear
-LIBS:regul
-LIBS:74xx
-LIBS:cmos4000
-LIBS:adc-dac
-LIBS:memory
-LIBS:xilinx
-LIBS:microcontrollers
-LIBS:dsp
-LIBS:microchip
-LIBS:analog_switches
-LIBS:motorola
-LIBS:texas
-LIBS:intel
-LIBS:audio
-LIBS:interface
-LIBS:digital-audio
-LIBS:philips
-LIBS:display
-LIBS:cypress
-LIBS:siliconi
-LIBS:opto
-LIBS:atmel
-LIBS:contrib
-LIBS:valves
-LIBS:ROMs
-LIBS:kickswitch-cache
-EELAYER 25 0
+EESchema Schematic File Version 4
+EELAYER 30 0
 EELAYER END
 $Descr A3 16535 11693
@@
 $EndDescr
 $Comp
-L ATMEGA328P-PU U3
+L kickswitch-rescue:ATMEGA328P-PU U3
 U 1 1 5B091313
 P 6100 3550
@@
 A17out
 $Comp
-L Crystal Y1
+L kickswitch-rescue:Crystal Y1
 U 1 1 5B092CDE
 P 9900 3100
@@
 $EndComp
 $Comp
-L C_Small C1
+L kickswitch-rescue:C_Small C1
 U 1 1 5B092DCA
 P 10250 3150
@@
 $EndComp
 $Comp
-L C_Small C2
+L kickswitch-rescue:C_Small C2
 U 1 1 5B092E01
 P 10050 3250
@@
 $EndComp
 $Comp
-L R R1
+L kickswitch-rescue:R R1
 U 1 1 5B093167
 P 6250 1750
@@
 $EndComp
 $Comp
-L D D1
+L kickswitch-rescue:D D1
 U 1 1 5B094007
 P 6250 1500
@@
 $EndComp
 $Comp
-L C_Small C3
+L kickswitch-rescue:C_Small C3
 U 1 1 5B094117
 P 9150 4900
@@
 A17_set
 $Comp
-L MC23C4100_socket U4
+L kickswitch-rescue:MC23C4100_socket U4
 U 1 1 5B09495B
 P 6450 7200
@@
 $EndComp
 $Comp
-L M27C160 U5
+L kickswitch-rescue:M27C160 U5
 U 1 1 5B095B63
 P 12050 7350
@@
 Text Label 5700 7600 0    60   ~ 0
 A16
-NoConn ~ 5850 8400
 Entry Wire Line
 	5550 5900 5650 6000
@@
 NoConn ~ 6350 8700
 $Comp
-L SN74LVC1G08 U1
+L kickswitch-rescue:SN74LVC1G08 U1
 U 1 1 5B0A16D2
 P 8200 1750
@@
 $EndComp
 $Comp
-L SN74LVC1G32 U2
+L kickswitch-rescue:SN74LVC1G32 U2
 U 1 1 5B0A2AA8
 P 10150 1850
@@
 $EndComp
 $Comp
-L Conn_02x10_Odd_Even J1
+L kickswitch-rescue:Conn_02x10_Odd_Even J1
 U 1 1 5B2D8C5D
 P 4350 6500
@@
 PD6
 $Comp
-L R_Network08 RN1
+L kickswitch-rescue:R_Network08 RN1
 U 1 1 5B3DCCF4
 P 9750 6300
@@
 $EndComp
 $Comp
-L R_Network09 RN2
+L kickswitch-rescue:R_Network09 RN2
 U 1 1 5B3DCD27
 P 9750 7300
@@
 Text Label 9500 7000 0    60   ~ 0
 A9
-Text Label 9500 7100 0    60   ~ 0
+Text Label 9450 7100 0    60   ~ 0
 A10
-Text Label 9500 7200 0    60   ~ 0
+Text Label 9450 7200 0    60   ~ 0
 A11
-Text Label 9500 7300 0    60   ~ 0
+Text Label 9450 7300 0    60   ~ 0
 A12
-Text Label 9500 7400 0    60   ~ 0
+Text Label 9450 7400 0    60   ~ 0
 A13
-Text Label 9500 7500 0    60   ~ 0
+Text Label 9450 7500 0    60   ~ 0
 A14
-Text Label 9500 7600 0    60   ~ 0
+Text Label 9450 7600 0    60   ~ 0
 A15
-Text Label 9500 7700 0    60   ~ 0
+Text Label 9450 7700 0    60   ~ 0
 A16
 Text Label 4650 6900 0    60   ~ 0
@@
 	7100 3400 9550 3400
 Wire Wire Line
-	10750 1850 10750 1850
-Wire Wire Line
 	7100 3500 10650 3500
 Wire Wire Line
 	7100 3600 10550 3600
 Wire Wire Line
-	9700 2950 10250 2950
+	9700 2950 9900 2950
 Wire Wire Line
 	9700 3050 9700 2950
@@
 	7100 3050 9700 3050
 Wire Wire Line
-	9700 3250 9950 3250
+	9700 3250 9900 3250
 Wire Wire Line
 	9700 3150 9700 3250
@@
 	10150 3250 10250 3250
 Wire Wire Line
-	5200 4650 5200 7000
+	5200 4650 5200 4750
 Wire Wire Line
 	10250 3250 10250 5150
@@
 Connection ~ 8550 5150
 Wire Wire Line
-	5200 1750 5200 2750
-Wire Wire Line
-	3850 1750 6100 1750
+	5200 1750 5200 2450
+Wire Wire Line
+	3850 1750 4950 1750
 Connection ~ 5200 2450
 Wire Wire Line
 	7100 3900 7500 3900
 Wire Wire Line
-	7500 1750 7500 5250
-Wire Wire Line
-	6400 1750 7500 1750
+	7500 1750 7500 3900
+Wire Wire Line
+	6400 1750 6500 1750
 Connection ~ 5200 1750
 Wire Wire Line
@@
 Wire Wire Line
 	9150 4600 9150 4800
-Connection ~ 9150 4600
-Wire Wire Line
-	2500 7700 5850 7700
 Wire Wire Line
 	2500 7700 2500 1250
@@
 	6350 5300 6350 5700
 Wire Wire Line
-	3850 5300 11950 5300
+	3850 5300 6350 5300
 Wire Wire Line
 	3850 1750 3850 5300
-Connection ~ 6450 8700
 Wire Wire Line
 	11950 5300 11950 5850
 Wire Wire Line
-	11950 8850 14250 8850
+	11950 8850 12050 8850
 Wire Wire Line
 	14250 8850 14250 5150
@@
 Wire Wire Line
 	7050 7500 7250 7500
-Wire Bus Line
-	7350 6100 7350 9000
 Wire Wire Line
 	12650 6150 12850 6150
@@
 Wire Bus Line
 	7350 9000 12950 9000
-Wire Bus Line
-	12950 9000 12950 6250
 Wire Wire Line
 	5850 6000 5650 6000
@@
 	5650 7600 5850 7600
 Wire Bus Line
-	5550 5600 5550 7500
-Wire Bus Line
 	5550 5600 11150 5600
-Wire Bus Line
-	11150 5600 11150 7650
 Wire Wire Line
 	11450 6150 11250 6150
@@
 	8800 1750 9550 1750
 Wire Wire Line
-	5600 1350 9950 1350
+	5600 1350 8000 1350
 Wire Wire Line
 	5600 1350 5600 1750
@@
 Connection ~ 5600 1750
 Wire Wire Line
-	14250 5150 5200 5150
-Wire Wire Line
-	10250 5150 8550 5150
+	14250 5150 10450 5150
+Wire Wire Line
+	10250 5150 9150 5150
 Wire Wire Line
 	8550 8700 6450 8700
@@
 	10450 2250 10450 5150
 Wire Wire Line
-	8000 2250 10450 2250
+	8000 2250 9950 2250
 Wire Wire Line
 	8000 2250 8000 1950
@@
 	4900 5000 4900 6700
 Wire Wire Line
-	9950 5300 9950 6900
+	9950 5300 9950 5900
 Connection ~ 9950 5300
 Connection ~ 9950 5900
-Wire Bus Line
-	9300 5600 9300 7600
 Wire Wire Line
 	9400 5900 9550 5900
@@
 Text Label 7100 3600 0    60   ~ 0
 A19_set
+Wire Wire Line
+	9900 2950 10250 2950
+Wire Wire Line
+	9900 3250 9950 3250
+Wire Wire Line
+	8550 5150 5200 5150
+Wire Wire Line
+	5200 2450 5200 2750
+Wire Wire Line
+	5200 1750 5600 1750
+Wire Wire Line
+	4950 1750 5200 1750
+Wire Wire Line
+	7500 3900 7500 4600
+Wire Wire Line
+	6500 1750 7500 1750
+Wire Wire Line
+	6000 1750 6100 1750
+Wire Wire Line
+	7500 4600 7500 5250
+Wire Wire Line
+	9150 5150 8550 5150
+Wire Wire Line
+	12050 8850 14250 8850
+Wire Wire Line
+	5200 4750 5200 5150
+Wire Wire Line
+	5600 1750 6000 1750
+Wire Wire Line
+	10450 5150 10250 5150
+Wire Wire Line
+	8000 1350 9950 1350
+Wire Wire Line
+	9950 2250 10450 2250
+Wire Wire Line
+	5200 5150 5200 7000
+Wire Wire Line
+	10950 5300 11950 5300
+Wire Wire Line
+	9950 5300 10950 5300
+Wire Wire Line
+	9950 5900 9950 6900
+Wire Wire Line
+	6350 5300 9950 5300
+$Comp
+L Connector_Generic:Conn_01x03 J2
+U 1 1 5E95C176
+P 4250 8000
+F 0 "J2" H 4168 7675 50  0000 C CNN
+F 1 "Conn_01x03" H 4168 7766 50  0000 C CNN
+F 2 "Pin_Headers:Pin_Header_Straight_1x03_Pitch2.54mm" H 4250 8000 50  0001 C CNN
+F 3 "~" H 4250 8000 50  0001 C CNN
+	1    4250 8000
+	-1   0    0    1
+$EndComp
+Wire Wire Line
+	2500 7700 4800 7700
+Wire Wire Line
+	4800 7700 4800 8000
+Wire Wire Line
+	4800 8000 4450 8000
+Wire Wire Line
+	4450 7900 5300 7900
+Wire Wire Line
+	5300 7900 5300 7700
+Wire Wire Line
+	5300 7700 5850 7700
+Wire Wire Line
+	5850 8400 5300 8400
+Wire Wire Line
+	5300 8400 5300 8100
+Wire Wire Line
+	5300 8100 4450 8100
+Wire Bus Line
+	7350 6100 7350 9000
+Wire Bus Line
+	12950 6250 12950 9000
+Wire Bus Line
+	5550 5600 5550 7500
+Wire Bus Line
+	11150 5600 11150 7650
+Wire Bus Line
+	9300 5600 9300 7600
 $EndSCHEMATC
